Commit message: modified commit

File: urdf/kobuki_view.urdf (robot description, URDF)
Before this commit: robot basic_kobuki, 6 links, 5 joints
Links:
- link base_link: geometry collision cylinder length=${0.083+0.020} radius=${0.354/2}

Commit message: README added and fixed URDF geometry

File: urdf/kobuki_view.urdf (robot description, URDF)
Before this commit: robot basic_kobuki, 6 links, 5 joints
Links:
- link base_link: geometry collision cylinder length=${0.083+0.020} radius=${0.354/2}; visual cylinder length=0.083 radius=${0.354/2}

Commit message: added kobuki mesh

File: urdf/kobuki_view.urdf (robot description, URDF)
Before this commit: robot basic_kobuki, 6 links, 5 joints
Links:
- removed link top_box_link
- removed link top_cylinder_link
- link base_link: geometry collision cylinder length=${0.083+0.020} radius=${0.354/2}; visual mesh filename=package://kobuki_kinematics/meshes/main_body.dae
Joints:
- removed joint top_box_joint
- removed joint top_cylinder_joint
